File: hardware/_restore_backup_2026-09-11T10-08-57-454/LimeSDR-Mini_2v4.kicad_pcb (KiCad board)
At the start: 8 copper layers, 91.7 x 88.7 mm, 430 parts, among them IC1 LMS7002M, IC10 LM75, IC11 DAC6311IDCK, IC12 M24128, IC13 LD39100PUR, IC14 LMZ20501SILR, IC15 W25Q128JVSIQ, IC16 AD5662, IC17 AS431, IC18 LD39100PUR, IC2 M24128, IC20 74LVC1G3157FZ4, IC3 SKY13411-374LF, IC4 SKY13411-374LF, IC5 LD39100PUR, IC6 LD39100PUR, IC7 LFE5U-45F-MG285, IC9 LMK00105, J10 PC104-Mainboard, J11 Conn_Coaxial, J13 Conn_Coaxial, J3 FPGA GPIO, J4 FPGA EGPIO (board edge), J5 FPGA JTAG (board edge), J7 U.FL/MMCX, J8 U.FL/MMCX, J9 FAN, T1 TC1-1-13M-45+, T2 TC1-1-13M-45+, T3 TC1-1-13M-45+, T4 TC1-1-13M-45+, U2 GRF5115, U3 GRF5115

Commit message: Adding project and lib fixing
Parts:
- U3: footprint spacelab2:QFN-16_GRF -> library:QFN-16_GRF
Changed lines of the file:
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@@
 		)
 		(embedded_fonts no)
-		(model "${KIPRJMOD}/library/GRF5115/3D/GRF5115.stp"
-			(offset
-				(xyz 0 0 0)
-			)
-			(scale
-				(xyz 1 1 1)
-			)
-			(rotate
-				(xyz 0 0 0)
-			)
-		)
-		(model "${KIPRJMOD}/library/3dmodels/GRF5115.stp"
-			(offset
-				(xyz 0 0 0)
-			)
-			(scale
-				(xyz 1 1 1)
-			)
-			(rotate
-				(xyz 0 0 0)
-			)
-		)
 	)
 	(footprint "Resistor_SMD:R_0402_1005Metric"
@@
 		)
 		(embedded_fonts no)
-		(model "${KIPRJMOD}/library/3dmodels/SSW-126-01-G-D.stp"
-			(offset
-				(xyz 43.25 -0.75 0)
-			)
-			(scale
-				(xyz 1 1 1)
-			)
-			(rotate
-				(xyz -90 -0 90)
-			)
-		)
-		(model "${KIPRJMOD}/library/3dmodels/SSW-126-01-G-D.stp"
-			(offset
-				(xyz 38.2 -0.75 0)
-			)
-			(scale
-				(xyz 1 1 1)
-			)
-			(rotate
-				(xyz -90 -0 90)
-			)
-		)
 	)
 	(footprint "Inductor_SMD:L_0402_1005Metric"
@@
 		)
 	)
-	(footprint "spacelab2:QFN-16_GRF"
+	(footprint "library:QFN-16_GRF"
 		(layer "F.Cu")
 		(at 116.0811 137.3586 -45)
@@
 		)
 		(property "Datasheet" ""
-			(at 0 0 135)
+			(at 0 0 315)
 			(layer "F.Fab")
 			(hide yes)
@@
 		)
 		(property "Description" ""
-			(at 0 0 135)
+			(at 0 0 315)
 			(layer "F.Fab")
 			(hide yes)
@@
 		)
 		(fp_text user "*"
-			(at -2.4638 -1 135)
+			(at -2.4638 -1 315)
 			(layer "F.SilkS")
 			(effects
@@
 		)
 		(fp_text user "*"
-			(at -1.1684 -1 135)
+			(at -1.1684 -1 315)
 			(layer "F.Fab")
 			(effects
@@
 		)
 		(embedded_fonts no)
-		(model "${KIPRJMOD}/library/GRF5115/3D/GRF5115.stp"
-			(offset
-				(xyz 0 0 0)
-			)
-			(scale
-				(xyz 1 1 1)
-			)
-			(rotate
-				(xyz 0 0 0)
-			)
-		)
-		(model "${KIPRJMOD}/library/3dmodels/GRF5115.stp"
-			(offset
-				(xyz 0 0 0)
-			)
-			(scale
-				(xyz 1 1 1)
-			)
-			(rotate
-				(xyz 0 0 0)
-			)
-		)
 	)
 	(footprint "LimeMicroAltiumLib_pcbLib:CAP0402"
@@
 		)
 		(property "Value" "Conn_Coaxial"
-			(at 4.73 -0.81 0)
+			(at 4.73 -0.81 180)
 			(layer "F.Fab")
 			(effects
@@
 		)
 		(fp_text user "${REFERENCE}"
-			(at -4.58 -2.98 0)
+			(at -4.58 -2.98 180)
 			(layer "F.Fab")
 			(effects
@@
 		)
 		(model "D:/Gamer/Downloads/LimeSDR-Mini-v2-main/LimeSDR-Mini-v2-main-kicad-new/library/3dmodels/3D-outline_00012857_B_step.stp"
-			(hide yes)
 			(offset
 				(xyz 8.45 0.1 3)
@@
 			)
 		)
-		(model "${KIPRJMOD}/library/CONMCX002-SMD/CONMCX002-SMD.step"
-			(hide yes)
-			(offset
-				(xyz 0 0 0)
-			)
-			(scale
-				(xyz 1 1 1)
-			)
-			(rotate
-				(xyz -90 -0 -0)
-			)
-		)
-		(model "/home/lucas/Documents/spacelab/explora/hardware/lib/133-3701-311.stp"
-			(hide yes)
-			(offset
-				(xyz 0 0 3)
-			)
-			(scale
-				(xyz 1 1 1)
-			)
-			(rotate
-				(xyz 90 -180 -0)
-			)
-		)
-		(model "${KIPRJMOD}/library/3dmodels/133-3701-311.stp"
-			(offset
-				(xyz 0 0 3)
-			)
-			(scale
-				(xyz 1 1 1)
-			)
-			(rotate
-				(xyz 90 -180 -0)
-			)
-		)
 	)
 	(footprint "Resistor_SMD:R_0402_1005Metric"
@@
 		)
 		(property "Value" "Conn_Coaxial"
-			(at 4.69 -0.76 0)
+			(at 4.69 -0.76 180)
 			(layer "F.Fab")
 			(effects
@@
 		)
 		(fp_text user "${REFERENCE}"
-			(at -4.53 -2.98 0)
+			(at -4.53 -2.98 180)
 			(layer "F.Fab")
 			(effects
@@
 		)
 		(model "D:/Gamer/Downloads/LimeSDR-Mini-v2-main/LimeSDR-Mini-v2-main-kicad-new/library/3dmodels/3D-outline_00012857_B_step.stp"
-			(hide yes)
 			(offset
 				(xyz 8.45 0.1 3)
@@
 			)
 		)
-		(model "${KIPRJMOD}/library/CONMCX002-SMD/CONMCX002-SMD.step"
-			(hide yes)
-			(offset
-				(xyz 0 0 0)
-			)
-			(scale
-				(xyz 1 1 1)
-			)
-			(rotate
-				(xyz -90 -0 -0)
-			)
-		)
-		(model "${KIPRJMOD}/library/3dmodels/133-3701-311.stp"
-			(offset
-				(xyz 0 0 3)
-			)
-			(scale
-				(xyz 1 1 1)
-			)
-			(rotate
-				(xyz 90 -180 -0)
-			)
-		)
